File: hardware_kicad/opa656_test.kicad_pcb (KiCad board)
At the start: 4 copper layers, 18 parts, among them J1 Conn_01x03, X1 opa656, X2 opa656

Commit message: Modifications Made
Other:
- board outline added: 67 x 17 mm
Changed lines of the file:
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@@
 		)
+	)
+	(gr_rect
+		(start 93.75 88.25)
+		(end 160.75 105.25)
+		(stroke
+			(width 0.05)
+			(type default)
+		)
+		(fill no)
+		(layer "Edge.Cuts")
 	)
 	(segment
@@
 		(polygon
 			(pts
-				(xy 93.991346 88.491346) (xy 160.491346 88.295758) (xy 160.491346 104.991346) (xy 94.230476 104.991346)
+				(xy 93.991346 88.491346) (xy 160.491346 88.5) (xy 160.491346 104.991346) (xy 94 105)
 			)
 		)
